Commit message: Proper indentation for my_robot.xacro

File: catkin_ws/src/my_robot/urdf/my_robot.xacro (robot description, xacro)
@@ -2,6 +2,5 @@
 <robot name="my_robot" xmlns:xacro="http://www.ros.org/wiki/xacro">
   <xacro:property name="caster_x_origin" value="0.225" />
-  <xacro:property name="front_wheel_hinge_joint_origin_x" value="0.15" />
-  <xacro:property name="back_wheel_hinge_joint_origin_x" value="-0.15" />
+  <xacro:property name="wheel_hinge_joint_origin_x" value="0.15" />
   <xacro:include filename="$(find my_robot)/urdf/my_robot.gazebo" />
   <link name="robot_footprint_1"></link>
@@ -34,213 +33,189 @@
       </geometry>
     </visual>
-    <collision name='back_caster_collision'>
-	    <origin xyz="-${caster_x_origin} 0 -0.05" rpy=" 0 0 0"/>
-      <geometry>
-        <sphere radius="0.0499"/>
-      </geometry>
-    </collision>
-    <visual name='back_caster_visual'>
-      <origin xyz="-${caster_x_origin} 0 -0.05" rpy=" 0 0 0"/>
-      <geometry>
-        <sphere radius="0.05"/>
-      </geometry>
-    </visual>
-    <collision name='front_caster_collision'>
-      <origin xyz="${caster_x_origin}  0 -0.05" rpy=" 0 0 0"/>
-      <geometry>
-        <sphere radius="0.0499"/>
-      </geometry>
-    </collision>
-    <visual name='front_caster_visual'>
-      <origin xyz="${caster_x_origin} 0 -0.05" rpy=" 0 0 0"/>
-      <geometry>
-        <sphere radius="0.05"/>
-      </geometry>
-    </visual>
   </link>
   <link name="front_left_wheel">
-	  <collision name="front_left_wheel_collision">
-		  <origin xyz="0 0 0" rpy=" 0 1.5707 1.5707"/>
-		  <geometry>
-			  <cylinder radius="0.1" length="0.05"/>
-		  </geometry>
-	  </collision>
-	  <inertial>
-		  <mass value="5"/>
-		  <origin xyz="0 0 0" rpy=" 0 1.5707 1.5707"/>
-		  <inertia
-			  ixx="0.1" ixy="0" ixz="0"
-			  iyy="0.1" iyz="0"
-			  izz="0.1"
-			  />
-	  </inertial>
-	  <visual name="front_left_wheel_visual">
-		  <origin xyz="0 0 0" rpy=" 0 1.5707 1.5707"/>
-		  <geometry>
-			  <cylinder radius="0.1" length="0.05"/>
-		  </geometry>
-	  </visual>
+    <collision name="front_left_wheel_collision">
+      <origin xyz="0 0 0" rpy=" 0 1.5707 1.5707"/>
+      <geometry>
+        <cylinder radius="0.1" length="0.05"/>
+      </geometry>
+    </collision>
+    <visual name="front_left_wheel_visual">
+      <origin xyz="0 0 0" rpy=" 0 1.5707 1.5707"/>
+      <geometry>
+        <cylinder radius="0.1" length="0.05"/>
+      </geometry>
+    </visual>
+    <inertial>
+      <mass value="5"/>
+	<origin xyz="0 0 0" rpy=" 0 1.5707 1.5707"/>
+	<inertia
+	  ixx="0.1" ixy="0" ixz="0"
+	  iyy="0.1" iyz="0"
+	  izz="0.1"
+	/>
+    </inertial>
+  </link>
+  <link name="front_right_wheel">
+    <collision name="front_right_wheel_collision">
+      <origin xyz="0 0 0" rpy=" 0 1.5707 1.5707"/>
+      <geometry>
+        <cylinder radius="0.1" length="0.05"/>
+      </geometry>
+    </collision>
+    <visual name="front_right_wheel_visual">
+      <origin xyz="0 0 0" rpy=" 0 1.5707 1.5707"/>
+      <geometry>
+        <cylinder radius="0.1" length="0.05"/>
+      </geometry>
+    </visual>
+    <inertial>
+      <mass value="5"/>
+      <origin xyz="0 0 0" rpy=" 0 1.5707 1.5707"/>
+      <inertia
+        ixx="0.1" ixy="0" ixz="0"
+        iyy="0.1" iyz="0"
+	izz="0.1"
+      />
+    </inertial>
+  </link>
+  <link name="back_left_wheel">
+    <collision name="back_left_wheel_collision">
+      <origin xyz="0 0 0" rpy=" 0 1.5707 1.5707"/>
+      <geometry>
+        <cylinder radius="0.1" length="0.05"/>
+      </geometry>
+    </collision>
+    <visual name="back_left_wheel_visual">
+      <origin xyz="0 0 0" rpy=" 0 1.5707 1.5707"/>
+      <geometry>
+        <cylinder radius="0.1" length="0.05"/>
+      </geometry>
+    </visual>
+    <inertial>
+      <mass value="5"/>
+      <origin xyz="0 0 0" rpy=" 0 1.5707 1.5707"/>
+      <inertia
+        ixx="0.1" ixy="0" ixz="0"
+	iyy="0.1" iyz="0"
+	izz="0.1"
+      />
+    </inertial>
+  </link>
+  <link name="back_right_wheel">
+    <collision name="back_right_wheel_collision">
+      <origin xyz="0 0 0" rpy=" 0 1.5707 1.5707"/>
+      <geometry>
+        <cylinder radius="0.1" length="0.05"/>
+      </geometry>
+    </collision>
+    <visual name="back_right_wheel_visual">
+      <origin xyz="0 0 0" rpy=" 0 1.5707 1.5707"/>
+      <geometry>
+        <cylinder radius="0.1" length="0.05"/>
+      </geometry>
+    </visual>
+    <inertial>
+      <mass value="5"/>
+      <origin xyz="0 0 0" rpy=" 0 1.5707 1.5707"/>
+      <inertia
+        ixx="0.1" ixy="0" ixz="0"
+	iyy="0.1" iyz="0"
+	izz="0.1"
+      />
+    </inertial>
   </link>
   <joint type="continuous" name="front_left_wheel_hinge">
-	  <origin xyz="${front_wheel_hinge_joint_origin_x} 0.175 0" rpy="0 0 0"/>
-	  <child link="front_left_wheel"/>
-	  <parent link="chassis"/>
-	  <axis xyz="0 1 0" rpy="0 0 0"/>
-	  <limit effort="10000" velocity="1000"/>
-	  <dynamics damping="1.0" friction="1.0"/>
-  </joint>
- <link name="front_right_wheel">
-	  <collision name="front_right_wheel_collision">
-		  <origin xyz="0 0 0" rpy=" 0 1.5707 1.5707"/>
-		  <geometry>
-			  <cylinder radius="0.1" length="0.05"/>
-		  </geometry>
-	  </collision>
-	  <inertial>
-		  <mass value="5"/>
-		  <origin xyz="0 0 0" rpy=" 0 1.5707 1.5707"/>
-		  <inertia
-			  ixx="0.1" ixy="0" ixz="0"
-			  iyy="0.1" iyz="0"
-			  izz="0.1"
-			  />
-	  </inertial>
-	  <visual name="front_right_wheel_visual">
-		  <origin xyz="0 0 0" rpy=" 0 1.5707 1.5707"/>
-		  <geometry>
-			  <cylinder radius="0.1" length="0.05"/>
-		  </geometry>
-	  </visual>
-  </link>
+    <origin xyz="${wheel_hinge_joint_origin_x} 0.175 0" rpy="0 0 0"/>
+    <child link="front_left_wheel"/>
+    <parent link="chassis"/>
+    <axis xyz="0 1 0" rpy="0 0 0"/>
+    <limit effort="10000" velocity="1000"/>
+    <dynamics damping="1.0" friction="1.0"/>
+  </joint>
   <joint type="continuous" name="front_right_wheel_hinge">
-	  <origin xyz="${front_wheel_hinge_joint_origin_x} -0.175 0" rpy="0 0 0"/>
-	  <child link="front_right_wheel"/>
-	  <parent link="chassis"/>
-	  <axis xyz="0 1 0" rpy="0 0 0"/>
-	  <limit effort="10000" velocity="1000"/>
-	  <dynamics damping="1.0" friction="1.0"/>
-  </joint>
-  <link name="back_left_wheel">
-	  <collision name="back_left_wheel_collision">
-		  <origin xyz="0 0 0" rpy=" 0 1.5707 1.5707"/>
-		  <geometry>
-			  <cylinder radius="0.1" length="0.05"/>
-		  </geometry>
-	  </collision>
-	  <inertial>
-		  <mass value="5"/>
-		  <origin xyz="0 0 0" rpy=" 0 1.5707 1.5707"/>
-		  <inertia
-			  ixx="0.1" ixy="0" ixz="0"
-			  iyy="0.1" iyz="0"
-			  izz="0.1"
-			  />
-	  </inertial>
-	  <visual name="back_left_wheel_visual">
-		  <origin xyz="0 0 0" rpy=" 0 1.5707 1.5707"/>
-		  <geometry>
-			  <cylinder radius="0.1" length="0.05"/>
-		  </geometry>
-	  </visual>
-  </link>
+    <origin xyz="${wheel_hinge_joint_origin_x} -0.175 0" rpy="0 0 0"/>
+    <child link="front_right_wheel"/>
+    <parent link="chassis"/>
+    <axis xyz="0 1 0" rpy="0 0 0"/>
+    <limit effort="10000" velocity="1000"/>
+    <dynamics damping="1.0" friction="1.0"/>
+  </joint>
   <joint type="continuous" name="back_left_wheel_hinge">
-	  <origin xyz="${back_wheel_hinge_joint_origin_x} 0.175 0" rpy="0 0 0"/>
-	  <child link="back_left_wheel"/>
-	  <parent link="chassis"/>
-	  <axis xyz="0 1 0" rpy="0 0 0"/>
-	  <limit effort="10000" velocity="1000"/>
-	  <dynamics damping="1.0" friction="1.0"/>
-  </joint>
- <link name="back_right_wheel">
-	  <collision name="back_right_wheel_collision">
-		  <origin xyz="0 0 0" rpy=" 0 1.5707 1.5707"/>
-		  <geometry>
-			  <cylinder radius="0.1" length="0.05"/>
-		  </geometry>
-	  </collision>
-	  <inertial>
-		  <mass value="5"/>
-		  <origin xyz="0 0 0" rpy=" 0 1.5707 1.5707"/>
-		  <inertia
-			  ixx="0.1" ixy="0" ixz="0"
-			  iyy="0.1" iyz="0"
-			  izz="0.1"
-			  />
-	  </inertial>
-	  <visual name="back_right_wheel_visual">
-		  <origin xyz="0 0 0" rpy=" 0 1.5707 1.5707"/>
-		  <geometry>
-			  <cylinder radius="0.1" length="0.05"/>
-		  </geometry>
-	  </visual>
-  </link>
+    <origin xyz="-${wheel_hinge_joint_origin_x} 0.175 0" rpy="0 0 0"/>
+    <child link="back_left_wheel"/>
+    <parent link="chassis"/>
+    <axis xyz="0 1 0" rpy="0 0 0"/>
+    <limit effort="10000" velocity="1000"/>
+    <dynamics damping="1.0" friction="1.0"/>
+  </joint>
   <joint type="continuous" name="back_right_wheel_hinge">
-	  <origin xyz="${back_wheel_hinge_joint_origin_x} -0.175 0" rpy="0 0 0"/>
-	  <child link="back_right_wheel"/>
-	  <parent link="chassis"/>
-	  <axis xyz="0 1 0" rpy="0 0 0"/>
-	  <limit effort="10000" velocity="1000"/>
-	  <dynamics damping="1.0" friction="1.0"/>
-  </joint>
-    <link name="camera">
-	  <inertial>
-		  <mass value="0.1"/>
-		  <origin xyz="0 0 0" rpy=" 0 0 0"/>
-		  <inertia
-			  ixx="1e-6" ixy="0" ixz="0"
-			  iyy="1e-6" iyz="0"
-			  izz="1e-6"
-			  />
-		  <box_inertia
-			  m="0.1" x="0.05" y="0.05" z="0.05"
-			  />
-	  </inertial>
-	  <collision name="camera_collision">
-		  <origin xyz="0 0 0" rpy=" 0 0 0"/>
-		  <geometry>
-			  <box size="0.05 0.05 0.05"/>
-		  </geometry>
-	  </collision>
-	  <visual name="camera_visual">
-		  <origin xyz="0 0 0" rpy=" 0 0 0"/>
-		  <geometry>
-			  <box size="0.05 0.05 0.05"/>
-		  </geometry>
-	  </visual>
+    <origin xyz="-${wheel_hinge_joint_origin_x} -0.175 0" rpy="0 0 0"/>
+    <child link="back_right_wheel"/>
+    <parent link="chassis"/>
+    <axis xyz="0 1 0" rpy="0 0 0"/>
+    <limit effort="10000" velocity="1000"/>
+    <dynamics damping="1.0" friction="1.0"/>
+  </joint>
+  <link name="camera">
+    <inertial>
+      <mass value="0.1"/>
+      <origin xyz="0 0 0" rpy=" 0 0 0"/>
+      <inertia
+        ixx="1e-6" ixy="0" ixz="0"
+        iyy="1e-6" iyz="0"
+        izz="1e-6"
+      />
+      <box_inertia
+        m="0.1" x="0.05" y="0.05" z="0.05"
+      />
+    </inertial>
+    <collision name="camera_collision">
+      <origin xyz="0 0 0" rpy=" 0 0 0"/>
+      <geometry>
+        <box size="0.05 0.05 0.05"/>
+      </geometry>
+    </collision>
+    <visual name="camera_visual">
+      <origin xyz="0 0 0" rpy=" 0 0 0"/>
+        <geometry>
+	  <box size="0.05 0.05 0.05"/>
+	</geometry>
+    </visual>
   </link>
   <joint type="fixed" name="camera_joint">
-	  <origin xyz="0.3 0 0" rpy=" 0 0 0"/>
-	  <axis xyz="0 1 0" />
-	  <child link="camera"/>
-	  <parent link="chassis"/>
+    <origin xyz="0.3 0 0" rpy=" 0 0 0"/>
+    <axis xyz="0 1 0" />
+    <child link="camera"/>
+    <parent link="chassis"/>
   </joint>
   <link name="hokuyo">
-	  <inertial>
-		  <mass value="1e-5"/>
-		  <origin xyz="0 0 0" rpy=" 0 0 0"/>
-		  <inertia
-			  ixx="1e-6" ixy="0" ixz="0"
-			  iyy="1e-6" iyz="0"
-			  izz="1e-6"
-			  />
-	  </inertial>
-	  <collision name="hokuyo_collision">
-		  <origin xyz="0 0 0" rpy=" 0 0 0"/>
-		  <geometry>
-			  <box size="0.1 0.1 0.1"/>
-		  </geometry>
-	  </collision>
-	  <visual name="hokuyo_visual">
-		  <origin xyz="0 0 0" rpy=" 0 0 0"/>
-		  <geometry>
-			  <mesh filename = "package://my_robot/meshes/hokuyo.dae"/>
-		  </geometry>
-	  </visual>
+    <inertial>
+      <mass value="1e-5"/>
+      <origin xyz="0 0 0" rpy=" 0 0 0"/>
+      <inertia
+        ixx="1e-6" ixy="0" ixz="0"
+        iyy="1e-6" iyz="0"
+        izz="1e-6"
+      />
+    </inertial>
+    <collision name="hokuyo_collision">
+      <origin xyz="0 0 0" rpy=" 0 0 0"/>
+      <geometry>
+        <box size="0.1 0.1 0.1"/>
+      </geometry>
+    </collision>
+    <visual name="hokuyo_visual">
+      <origin xyz="0 0 0" rpy=" 0 0 0"/>
+      <geometry>
+        <mesh filename = "package://my_robot/meshes/hokuyo.dae"/>
+      </geometry>
+    </visual>
   </link>
   <joint type="fixed" name="hokuyo_joint">
-	  <origin xyz="0.25 0 0.075" rpy=" 0 0 0"/>
-	  <axis xyz="0 1 0" rpy=" 0 0 0"/>
-	  <child link="hokuyo"/>
-	  <parent link="chassis"/>
-   </joint>
+    <origin xyz="0.25 0 0.075" rpy=" 0 0 0"/>
+    <axis xyz="0 1 0" rpy=" 0 0 0"/>
+    <child link="hokuyo"/>
+    <parent link="chassis"/>
+  </joint>
 </robot>
